File: Audio.kicad_sch (KiCad schematic)
At the start: 51 parts, among them J14 Conn_01x06_Socket, J19 Conn_01x06_Pin, U1 TL072, U10 TL072, U11 TL072

Commit message: Tweaks to pcb, regenerated gerber
Parts:
- VR1: footprint PCM_4ms_Potentiometer:Bourns_3362 -> Potentiometer_THT:Potentiometer_Bourns_3296W_Vertical
Changed lines of the file:
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@@
       (effects (font (size 1.27 1.27)))
     )
-    (property "Footprint" "PCM_4ms_Potentiometer:Bourns_3362" (at 215.9 52.07 0)
+    (property "Footprint" "Potentiometer_THT:Potentiometer_Bourns_3296W_Vertical" (at 215.9 52.07 0)
       (effects (font (size 1.27 1.27)) (justify left) hide)
     )
