File: summer.kicad_pcb (KiCad board)
At the start: 2 copper layers, 135.6 x 83.1 mm, 145 parts, among them J1 AudioJack3_Switch, J10 Conn_01x02_Socket, J11 Conn_01x06_Socket, J12 Conn_01x03_Socket, J14 Conn_01x06_Socket, J15 Conn_01x07_Socket, J16 Conn_01x04_Socket, J2 AudioJack2_Switch, J23 Conn_01x06, J24 Conn_01x06, J3 AudioJack2_Switch, J4 AudioJack2, J5 Mag_Pre_Send, J6 Mag_Pre_Return, J7 Piezo_Pre_Send, J8 Piezo_Pre_Return, J9 AudioJack2, K1 TQ-2-5V, K2 TQ-2-5V, K3 TQ-2-5V, SW1 SW_Push_DPDT, SW2 SW_Push_DPDT, SW3 3PDTBLUE, U1 L78L05_TO92, U10 TLP222A, U11 7400, U12 74HCT74, U13 74HCT4075, U14 74HCT11, U15 74HCT14, U2 TL072, U3 TL072, U4 TL072, U5 MV57, U6 MV57, U7 MV57, U8 TLP222A, U9 TLP222A

Commit message: Tweaks to pcb, regenerated gerber
Parts:
- VR1: footprint PCM_4ms_Potentiometer:Bourns_3362 -> Potentiometer_THT:Potentiometer_Bourns_3296W_Vertical
- moved C24 14.2 mm to (-82.2, 22.9), turned to 0 degrees
- moved VR1 3.64 mm to (-3.56, -29.2)
- moved C4 2.36 mm to (-64.3, -13.2)
- moved C5 1.61 mm to (-53.1, 7.62)
- moved U1 1.33 mm to (-57.4, 7.62)
- moved C6 1.05 mm to (-62.5, 2.54)
- moved D2 1.05 mm to (-63.0, -0.51)
- moved J12 0.76 mm to (-80.0, 15.0)
- moved C12 0.57 mm to (32.8, -27.7)
- moved C20 0.25 mm to (5.63, -29.5)
Routing:
- net Net-(U7-GP5): track 70.5 -> 84.9 mm
- net GNDD: track 175.6 -> 169.3 mm
- net GNDPWR: track 76.6 -> 82.5 mm
- net Net-(U4A--): track 31.8 -> 28.1 mm
- net Net-(VR1-S): track 6.23 -> 8.26 mm
- net Vref: track 140.6 -> 139.3 mm
- net +9V: track 239.2 -> 240.3 mm
- net /Switching/MAG_LED_ON: track 18.4 -> 17.6 mm
